File: Assignment1/Assignment1.kicad_sch (KiCad schematic)
At the start: 4 parts, among them SW1 SW_SPST

Commit message: Finished
Parts:
- SW1: footprint Button_Switch_SMD:SW_Push_1P1T_NO_6x6mm_H9.5mm -> Button_Switch_THT:SW_PUSH_6mm
Changed lines of the file:
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@@
       (effects (font (size 1.27 1.27)) (justify left))
     )
-    (property "Footprint" "Button_Switch_SMD:SW_Push_1P1T_NO_6x6mm_H9.5mm" (at 111.76 81.28 0)
+    (property "Footprint" "Button_Switch_THT:SW_PUSH_6mm" (at 111.76 81.28 0)
       (effects (font (size 1.27 1.27)) hide)
     )
